Commit message: Use default world instead, fix laser z position

File: csl_robot_descriptions/defs/hokuyo_laser.xacro (robot description, xacro)
@@ -5,5 +5,5 @@
         <joint name="hokuyo_joint" type="fixed">
             <axis xyz="0 1 0" />
-            <origin xyz="0.0 0.0 0.0" rpy="0 0 0"/>
+            <origin xyz="0.0 0.0 ${hokuyo_height/4}" rpy="0 0 0"/>
             <parent link="top_plate"/>
             <child link="hokuyo_link"/>

Commit message: Add to the gazebo simulation setup

File: csl_robot_descriptions/defs/hokuyo_laser.xacro (robot description, xacro)
@@ -1,9 +1,9 @@
 <?xml version="1.0"?>
 <robot xmlns:xacro="http://ros.org/wiki/xacro" >
-    <xacro:property name="hokuyo_height" value="0.1" />
+    <xacro:property name="hokuyo_size" value="0.1" />
     <xacro:macro name="hokuyo_laser">
         <joint name="hokuyo_joint" type="fixed">
             <axis xyz="0 1 0" />
-            <origin xyz="0.0 0.0 ${hokuyo_height/4}" rpy="0 0 0"/>
+            <origin xyz="0.0 0.0 ${hokuyo_size/4}" rpy="0 0 0"/>
             <parent link="top_plate"/>
             <child link="hokuyo_link"/>
@@ -14,5 +14,5 @@
                 <origin xyz="0 0 0" rpy="0 0 0"/>
                 <geometry>
-                    <box size="0.1 0.1 0.1"/>
+                    <box size="${hokuyo_size} ${hokuyo_size} ${hokuyo_size}"/>
                 </geometry>
             </collision>
@@ -22,4 +22,5 @@
                     <mesh filename="package://csl_robot_descriptions/meshes/hokuyo.dae"/>
                 </geometry>
+                <material name="black"/>
             </visual>
             <inertial>
@@ -29,4 +30,7 @@
             </inertial>
         </link>
+	    <gazebo reference="hokuyo_link">
+		    <material value="Gazebo/Black"/>
+	    </gazebo>
         <!-- Hokuyo Laser -->
         <gazebo reference="hokuyo_link">
@@ -63,5 +67,5 @@
                 </ray>
                 <plugin name="gazebo_ros_head_hokuyo_controller" filename="libgazebo_ros_gpu_laser.so">
-                    <topicName>/rrbot/laser/scan</topicName>
+                    <topicName>scan</topicName>
                     <frameName>hokuyo_link</frameName>
                 </plugin>

File: csl_robot_descriptions/defs/pioneer3at.xacro (robot description, xacro)
@@ -6,4 +6,5 @@
     name="pioneer_3at">
     <xacro:include filename="$(find csl_robot_descriptions)/defs/pioneer3at_body.xacro"/>
+    <xacro:chassis />
     <xacro:p3at_front suffix="left" reflect="1"/>
     <xacro:p3at_front suffix="right" reflect="-1"/>
@@ -13,3 +14,7 @@
     <xacro:include filename="$(find csl_robot_descriptions)/defs/hokuyo_laser.xacro"/>
     <xacro:hokuyo_laser/>
+    <xacro:include filename="$(find csl_robot_descriptions)/defs/camera.xacro"/>
+    <xacro:camera_macro camera_name="$(arg camera_name)"/>
+    <!--<xacro:include filename="$(find csl_robot_descriptions)/defs/marker.xacro"/>-->
+    <!--<xacro:ar_sys_marker parent="top_plate" marker_id="1" /> -->
 </robot>

File: csl_robot_descriptions/defs/pioneer3at_body.xacro (robot description, xacro)
@@ -6,127 +6,129 @@
     >
     <!-- Chassis -->
-	<link name="base_link">
-		<inertial>
-			<mass value="10.0"/>
-			<origin xyz="0 0 0.177"/>
-			<inertia ixx="0.3338" ixy="0.0" ixz="0.0"
-				iyy="0.4783" iyz="0.0"
-				izz="0.3338"/>
-		</inertial>
-		<visual name="base_visual">
-			<origin xyz="0 0 0.177" rpy="0 0 0"/>
-			<geometry name="pioneer_geom">
-				<mesh filename="package://p2os_urdf/meshes/p3at_meshes/chassis.stl"/>
-			</geometry>
-			<material name="ChassisRed">
-				<color rgba="0.851 0.0 0.0 1.0"/>
-			</material>
-		</visual>
-		<collision>
-			<origin xyz="0 0 0.177" rpy="0 0 0"/>
-			<geometry>
-				<mesh filename="package://p2os_urdf/meshes/p3at_meshes/chassis.stl"/>
-			</geometry>
-		</collision>
-	</link>
-	<gazebo reference="base_link">
-		<material value="Gazebo/Red"/>
-	</gazebo>
-    <!-- Top -->
-	<link name="top_plate">
-		<inertial>
-			<mass value="0.1"/>
-			<origin xyz="-0.025 0 -0.223"/>
-			<inertia ixx="1.0" ixy="0.0" ixz="0.0"
-				iyy="1.0" iyz="0.0"
- 				izz="1.0"/>
-		</inertial>
-		<visual name="base_visual">
-			<origin xyz="0 0 0" rpy="0 0 0"/>
-			<geometry name="pioneer_geom">
-				<mesh filename="package://p2os_urdf/meshes/p3at_meshes/top.stl"/>
-			</geometry>
-			<material name="TopBlack">
-				<color rgba="0.038 0.038 0.038 1.0"/>
-			</material>
-		</visual>
-		<collision>
-			<origin xyz="0 0 0" rpy="0 0 0"/>
-			<geometry>
-				<box size="0 0 0"/>
-			</geometry>
-		</collision>
-	</link>
-	<gazebo reference="top_plate">
-		<material value="Gazebo/Black"/>
-	</gazebo>
-	<joint name="base_top_joint" type="fixed">
-		<origin xyz="0.003 0 0.274" rpy="0 0 0"/>
-		<parent link="base_link"/>
-		<child link="top_plate"/>
-	</joint>
-    <!-- Front + Back Sonar -->
-	<link name="front_sonar">
-		<inertial>
-			<mass value="0.1"/>
-			<origin xyz="0 0 0"/>
-			<inertia ixx="1.0" ixy="0.0" ixz="0.0"
-				iyy="1.0" iyz="0.0" izz="1.0"/>
-		</inertial>
-		<visual name="base_visual">
-			<origin xyz="0 0 0" rpy="0 0 0"/>
-			<geometry name="pioneer_geom">
-				<mesh filename="package://p2os_urdf/meshes/p3at_meshes/front_sonar.stl"/>
-			</geometry>
-			<material name="SonarYellow">
-				<color rgba="0.715 0.583 0.210 1.0"/>
-			</material>
-		</visual>
-		<collision>
-			<origin xyz="0 0 0" rpy="0 0 0"/>
-			<geometry>
-				<box size="0 0 0"/>
-			</geometry>
-		</collision>
-	</link>
-	<gazebo reference="front_sonar">
-		<material value="Gazebo/Yellow"/>
-	</gazebo>
-	<joint name="base_front_joint" type="fixed">
-		<origin xyz="0.193 0 0.25" rpy="0 0 0"/>
-		<parent link="base_link"/>
-		<child link="front_sonar"/>
-	</joint>
-	<link name="back_sonar">
-		<inertial>
-			<mass value="0.1"/>
-			<origin xyz="0 0 0"/>
-			<inertia ixx="1.0" ixy="0.0" ixz="0.0"
-				iyy="1.0" iyz="0.0" izz="1.0"/>
-		</inertial>
-		<visual name="base_visual">
-			<origin xyz="0 0 0" rpy="0 0 0"/>
-			<geometry name="pioneer_geom">
-				<mesh filename="package://p2os_urdf/meshes/p3at_meshes/back_sonar.stl"/>
-			</geometry>
-			<material name="SonarYellow">
-				<color rgba="0.715 0.583 0.210 1.0"/>
-			</material>
-		</visual>
-		<collision>
-			<origin xyz="0 0 0" rpy="0 0 0"/>
-			<geometry>
-				<box size="0 0 0"/>
-			</geometry>
-		</collision>
-	</link>
-	<gazebo reference="back_sonar">
-		<material value="Gazebo/Yellow"/>
-	</gazebo>
-	<joint name="base_back_joint" type="fixed">
-		<origin xyz="-0.187 0 0.247" rpy="0 0 0"/>
-		<parent link="base_link"/>
-		<child link="back_sonar"/>
-	</joint>
+    <xacro:macro name="chassis">
+	    <link name="base_link">
+		    <inertial>
+			    <mass value="10.0"/>
+			    <origin xyz="0 0 0.177"/>
+			    <inertia ixx="0.3338" ixy="0.0" ixz="0.0"
+				    iyy="0.4783" iyz="0.0"
+				    izz="0.3338"/>
+		    </inertial>
+		    <visual name="base_visual">
+			    <origin xyz="0 0 0.177" rpy="0 0 0"/>
+			    <geometry name="pioneer_geom">
+				    <mesh filename="package://p2os_urdf/meshes/p3at_meshes/chassis.stl"/>
+			    </geometry>
+			    <material name="ChassisRed">
+				    <color rgba="0.851 0.0 0.0 1.0"/>
+			    </material>
+		    </visual>
+		    <collision>
+			    <origin xyz="0 0 0.177" rpy="0 0 0"/>
+			    <geometry>
+				    <mesh filename="package://p2os_urdf/meshes/p3at_meshes/chassis.stl"/>
+			    </geometry>
+		    </collision>
+	    </link>
+	    <gazebo reference="base_link">
+		    <material value="Gazebo/Red"/>
+	    </gazebo>
+        <!-- Top -->
+	    <link name="top_plate">
+		    <inertial>
+			    <mass value="0.1"/>
+			    <origin xyz="-0.025 0 -0.223"/>
+			    <inertia ixx="1.0" ixy="0.0" ixz="0.0"
+				    iyy="1.0" iyz="0.0"
+ 				    izz="1.0"/>
+		    </inertial>
+		    <visual name="base_visual">
+			    <origin xyz="0 0 0" rpy="0 0 0"/>
+			    <geometry name="pioneer_geom">
+				    <mesh filename="package://p2os_urdf/meshes/p3at_meshes/top.stl"/>
+			    </geometry>
+			    <material name="TopBlack">
+				    <color rgba="0.038 0.038 0.038 1.0"/>
+			    </material>
+		    </visual>
+		    <collision>
+			    <origin xyz="0 0 0" rpy="0 0 0"/>
+			    <geometry>
+				    <box size="0 0 0"/>
+			    </geometry>
+		    </collision>
+	    </link>
+	    <gazebo reference="top_plate">
+		    <material value="Gazebo/Black"/>
+	    </gazebo>
+	    <joint name="base_top_joint" type="fixed">
+		    <origin xyz="0.003 0 0.274" rpy="0 0 0"/>
+		    <parent link="base_link"/>
+		    <child link="top_plate"/>
+	    </joint>
+        <!-- Front + Back Sonar -->
+	    <link name="front_sonar">
+		    <inertial>
+			    <mass value="0.1"/>
+			    <origin xyz="0 0 0"/>
+			    <inertia ixx="1.0" ixy="0.0" ixz="0.0"
+				    iyy="1.0" iyz="0.0" izz="1.0"/>
+		    </inertial>
+		    <visual name="base_visual">
+			    <origin xyz="0 0 0" rpy="0 0 0"/>
+			    <geometry name="pioneer_geom">
+				    <mesh filename="package://p2os_urdf/meshes/p3at_meshes/front_sonar.stl"/>
+			    </geometry>
+			    <material name="SonarYellow">
+				    <color rgba="0.715 0.583 0.210 1.0"/>
+			    </material>
+		    </visual>
+		    <collision>
+			    <origin xyz="0 0 0" rpy="0 0 0"/>
+			    <geometry>
+				    <box size="0 0 0"/>
+			    </geometry>
+		    </collision>
+	    </link>
+	    <gazebo reference="front_sonar">
+		    <material value="Gazebo/Yellow"/>
+	    </gazebo>
+	    <joint name="base_front_joint" type="fixed">
+		    <origin xyz="0.193 0 0.25" rpy="0 0 0"/>
+		    <parent link="base_link"/>
+		    <child link="front_sonar"/>
+	    </joint>
+	    <link name="back_sonar">
+		    <inertial>
+			    <mass value="0.1"/>
+			    <origin xyz="0 0 0"/>
+			    <inertia ixx="1.0" ixy="0.0" ixz="0.0"
+				    iyy="1.0" iyz="0.0" izz="1.0"/>
+		    </inertial>
+		    <visual name="base_visual">
+			    <origin xyz="0 0 0" rpy="0 0 0"/>
+			    <geometry name="pioneer_geom">
+				    <mesh filename="package://p2os_urdf/meshes/p3at_meshes/back_sonar.stl"/>
+			    </geometry>
+			    <material name="SonarYellow">
+				    <color rgba="0.715 0.583 0.210 1.0"/>
+			    </material>
+		    </visual>
+		    <collision>
+			    <origin xyz="0 0 0" rpy="0 0 0"/>
+			    <geometry>
+				    <box size="0 0 0"/>
+			    </geometry>
+		    </collision>
+	    </link>
+	    <gazebo reference="back_sonar">
+		    <material value="Gazebo/Yellow"/>
+	    </gazebo>
+	    <joint name="base_back_joint" type="fixed">
+		    <origin xyz="-0.187 0 0.247" rpy="0 0 0"/>
+		    <parent link="base_link"/>
+		    <child link="back_sonar"/>
+	    </joint>
+    </xacro:macro>
     <!-- Front Axles + Wheels + Hubcaps -->
     <xacro:macro name="p3at_front" params="suffix reflect">
