Commit message: WIP: Work towards mr-slam

File: csl_robot_descriptions/defs/hokuyo_laser.xacro (robot description, xacro)
@@ -63,5 +63,6 @@
                         -->
                         <mean>0.0</mean>
-                        <stddev>0.01</stddev>
+                        <!--<stddev>0.01</stddev>-->
+                        <stddev>0.1</stddev>
                     </noise>
                 </ray>

File: csl_robot_descriptions/defs/pioneer_3at_body.xacro (robot description, xacro)
@@ -1,371 +1,371 @@
 <?xml version="1.0"?>
 <robot xmlns:sensor="http://playerstage.sourceforge.net/gazebo/xmlschema/#sensor"
-    xmlns:controller="http://playerstage.sourceforge.net/gazebo/xmlschema/#controller"
-    xmlns:interface="http://playerstage.sourceforge.net/gazebo/xmlschema/#interface"
-    xmlns:xacro="http://ros.org/wiki/xacro"
-    >
-    <!-- Chassis -->
-    <xacro:macro name="chassis">
-	    <link name="base_link">
-		    <inertial>
-			    <mass value="10.0"/>
-			    <origin xyz="0 0 0.177"/>
-			    <inertia ixx="0.3338" ixy="0.0" ixz="0.0"
-				    iyy="0.4783" iyz="0.0"
-				    izz="0.3338"/>
-		    </inertial>
-		    <visual name="base_visual">
-			    <origin xyz="0 0 0.177" rpy="0 0 0"/>
-			    <geometry name="pioneer_geom">
-				    <mesh filename="package://p2os_urdf/meshes/p3at_meshes/chassis.stl"/>
-			    </geometry>
-			    <material name="ChassisRed">
-				    <color rgba="0.851 0.0 0.0 1.0"/>
-			    </material>
-		    </visual>
-		    <collision>
-			    <origin xyz="0 0 0.177" rpy="0 0 0"/>
-			    <geometry>
-				    <mesh filename="package://p2os_urdf/meshes/p3at_meshes/chassis.stl"/>
-			    </geometry>
-		    </collision>
-	    </link>
-	    <gazebo reference="base_link">
-		    <material value="Gazebo/Red"/>
-	    </gazebo>
-        <!-- Top -->
-	    <link name="top_plate">
-		    <inertial>
-			    <mass value="0.1"/>
-			    <origin xyz="-0.025 0 -0.223"/>
-			    <inertia ixx="1.0" ixy="0.0" ixz="0.0"
-				    iyy="1.0" iyz="0.0"
- 				    izz="1.0"/>
-		    </inertial>
-		    <visual name="base_visual">
-			    <origin xyz="0 0 0" rpy="0 0 0"/>
-			    <geometry name="pioneer_geom">
-				    <mesh filename="package://p2os_urdf/meshes/p3at_meshes/top.stl"/>
-			    </geometry>
-			    <material name="TopBlack">
-				    <color rgba="0.038 0.038 0.038 1.0"/>
-			    </material>
-		    </visual>
-		    <collision>
-			    <origin xyz="0 0 0" rpy="0 0 0"/>
-			    <geometry>
-				    <box size="0 0 0"/>
-			    </geometry>
-		    </collision>
-	    </link>
-	    <gazebo reference="top_plate">
-		    <material value="Gazebo/Black"/>
-	    </gazebo>
-	    <joint name="base_top_joint" type="fixed">
-		    <origin xyz="0.003 0 0.274" rpy="0 0 0"/>
-		    <parent link="base_link"/>
-		    <child link="top_plate"/>
-	    </joint>
-        <!-- Front + Back Sonar -->
-	    <link name="front_sonar">
-		    <inertial>
-			    <mass value="0.1"/>
-			    <origin xyz="0 0 0"/>
-			    <inertia ixx="1.0" ixy="0.0" ixz="0.0"
-				    iyy="1.0" iyz="0.0" izz="1.0"/>
-		    </inertial>
-		    <visual name="base_visual">
-			    <origin xyz="0 0 0" rpy="0 0 0"/>
-			    <geometry name="pioneer_geom">
-				    <mesh filename="package://p2os_urdf/meshes/p3at_meshes/front_sonar.stl"/>
-			    </geometry>
-			    <material name="SonarYellow">
-				    <color rgba="0.715 0.583 0.210 1.0"/>
-			    </material>
-		    </visual>
-		    <collision>
-			    <origin xyz="0 0 0" rpy="0 0 0"/>
-			    <geometry>
-				    <box size="0 0 0"/>
-			    </geometry>
-		    </collision>
-	    </link>
-	    <gazebo reference="front_sonar">
-		    <material value="Gazebo/Yellow"/>
-	    </gazebo>
-	    <joint name="base_front_joint" type="fixed">
-		    <origin xyz="0.193 0 0.25" rpy="0 0 0"/>
-		    <parent link="base_link"/>
-		    <child link="front_sonar"/>
-	    </joint>
-	    <link name="back_sonar">
-		    <inertial>
-			    <mass value="0.1"/>
-			    <origin xyz="0 0 0"/>
-			    <inertia ixx="1.0" ixy="0.0" ixz="0.0"
-				    iyy="1.0" iyz="0.0" izz="1.0"/>
-		    </inertial>
-		    <visual name="base_visual">
-			    <origin xyz="0 0 0" rpy="0 0 0"/>
-			    <geometry name="pioneer_geom">
-				    <mesh filename="package://p2os_urdf/meshes/p3at_meshes/back_sonar.stl"/>
-			    </geometry>
-			    <material name="SonarYellow">
-				    <color rgba="0.715 0.583 0.210 1.0"/>
-			    </material>
-		    </visual>
-		    <collision>
-			    <origin xyz="0 0 0" rpy="0 0 0"/>
-			    <geometry>
-				    <box size="0 0 0"/>
-			    </geometry>
-		    </collision>
-	    </link>
-	    <gazebo reference="back_sonar">
-		    <material value="Gazebo/Yellow"/>
-	    </gazebo>
-	    <joint name="base_back_joint" type="fixed">
-		    <origin xyz="-0.187 0 0.247" rpy="0 0 0"/>
-		    <parent link="base_link"/>
-		    <child link="back_sonar"/>
-	    </joint>
-    </xacro:macro>
-    <!-- Front Axles + Wheels + Hubcaps -->
-    <xacro:macro name="p3at_front" params="suffix reflect">
-	    <link name="p3at_front_${suffix}_axle">
-		    <inertial>
-			    <mass value="0.1"/>
-			    <origin xyz="0 0 0"/>
-			    <inertia ixx="1.0" ixy="0.0" ixz="0.0"
-				    iyy="1.0" iyz="0.0" izz="1.0"/>
-  	 	    </inertial>
-	        <visual name="base_visual">
-		        <origin xyz="0 0 0" rpy="0 0 0"/>
-		        <geometry name="pioneer_geom">
-			        <mesh filename="package://p2os_urdf/meshes/p3at_meshes/axle.stl"/>
-		        </geometry>
-		        <material name="AxleGrey">
-			        <color rgba="0.5 0.5 0.5 1"/>
-		        </material>
-	        </visual>
-	        <collision>
-		        <origin xyz="0 0 0" rpy="0 0 0"/>
-		        <geometry>
-			        <box size="0 0 0"/>
-		        </geometry>
-	        </collision>
-	    </link>
-	    <gazebo reference="p3at_front_${suffix}_axle">
-		    <material value="Gazebo/Grey"/>
-	    </gazebo>
-	    <joint name="base_front_${suffix}_axle_joint" type="fixed">
-		    <origin xyz="0.135 ${reflect*0.156} 0.111" rpy="0 0 0"/>
-		    <parent link="base_link"/>
-		    <child link="p3at_front_${suffix}_axle"/>
-	    </joint>
-	    <link name="p3at_front_${suffix}_hub">
-		    <inertial>
-			    <mass value="0.1"/>
-			    <origin xyz="0 0 0"/>
-			    <inertia ixx="1.0" ixy="0.0" ixz="0.0"
-				    iyy="1.0" iyz="0.0" izz="1.0"/>
-  	 	    </inertial>
-	        <visual name="base_visual">
-		        <origin xyz="0 0 0" rpy="0 0 0"/>
-		        <geometry name="pioneer_geom">
-			        <mesh filename="package://p2os_urdf/meshes/p3at_meshes/${suffix}_hubcap.stl"/>
-		        </geometry>
-		        <material name="HubcapYellow">
-			        <color rgba="1.0 0.811 0.151 1.0"/>
-		        </material>
-	        </visual>
-	        <collision>
-		        <origin xyz="0 0 0" rpy="0 0 0"/>
-		        <geometry>
-			        <box size="0 0 0"/>
-		        </geometry>
-	        </collision>
-	    </link>
-	    <gazebo reference="p3at_front_${suffix}_hub">
-		    <material value="Gazebo/Yellow"/>
-	    </gazebo>
-	    <joint name="base_front_${suffix}_hub_joint" type="fixed">
-		    <origin xyz="0 ${reflect*0.041} 0" rpy="0 0 0"/>
-		    <parent link="p3at_front_${suffix}_axle"/>
-		    <child link="p3at_front_${suffix}_hub"/>
-	    </joint>
-	    <link name="p3at_front_${suffix}_wheel">
-		    <inertial>
-			    <mass value="0.5"/>
-			    <origin xyz="0 0 0"/>
-			    <inertia ixx="0.012411765597" ixy="0" ixz="0"
-                    iyy="0.015218160428" iyz="0" izz="0.011763977943"/>
-            </inertial>
-	        <visual name="base_visual">
-		        <origin xyz="0 0 0" rpy="0 0 0"/>
-		        <geometry name="pioneer_geom">
-			        <mesh filename="package://p2os_urdf/meshes/p3at_meshes/wheel.stl"/>
-		        </geometry>
-		        <material name="WheelBlack">
-			        <color rgba="0.117 0.117 0.117 1"/>
-		        </material>
-	        </visual>
-	        <collision>
-		        <origin xyz="0 0 0" rpy="${-3.1415927/2} 0 0"/>
-		        <geometry>
-	                <!--mesh filename="package://p2os_urdf/meshes/p3at_meshes/wheel.stl"/-->
-	                <cylinder radius="0.111" length="0.075"/>
-		        </geometry>
-	        </collision>
-	    </link>
-	    <gazebo reference="p3at_front_${suffix}_wheel">
-		    <material value="Gazebo/Black"/>
-	    </gazebo>
-	    <joint name="p3at_front_${suffix}_wheel_joint" type="continuous">
-  	        <axis xyz="0 1 0"/>
-            <anchor xyz="0 0 0"/>
-            <limit effort="100" velocity="100" />
-            <joint_properties damping="0.7"/>
-		    <origin xyz="0 0 0" rpy="0 0 0"/>
-		    <parent link="p3at_front_${suffix}_hub"/>
-		    <child link="p3at_front_${suffix}_wheel"/>
-	    </joint>
-    </xacro:macro>
-    <!-- Back Axles + Wheels + Hubcaps -->
-    <xacro:macro name="p3at_back" params="suffix reflect">
-	    <link name="p3at_back_${suffix}_axle">
-		    <inertial>
-			    <mass value="0.1"/>
-			    <origin xyz="0 0 0"/>
-			    <inertia ixx="1.0" ixy="0.0" ixz="0.0"
-				    iyy="1.0" iyz="0.0" izz="1.0"/>
-  	 	    </inertial>
-	        <visual name="base_visual">
-		        <origin xyz="0 0 0" rpy="0 0 0"/>
-		        <geometry name="pioneer_geom">
-			        <mesh filename="package://p2os_urdf/meshes/p3at_meshes/axle.stl"/>
-		        </geometry>
-		        <material name="AxleGrey">
-			        <color rgba="0.5 0.5 0.5 1"/>
-		        </material>
-	        </visual>
-	        <collision>
-		        <origin xyz="0 0 0" rpy="0 0 0"/>
-		        <geometry>
-			        <mesh filename="package://p2os_urdf/meshes/p3at_meshes/axle.stl"/>
-		        </geometry>
-	        </collision>
-	    </link>
-	    <gazebo reference="p3at_back_${suffix}_axle">
-		    <material value="Gazebo/Grey"/>
-	    </gazebo>
-	    <joint name="bp3at_back_${suffix}_axle_joint" type="fixed">
-		    <origin xyz="-0.134 ${reflect*0.156} 0.111" rpy="0 0 0"/>
-		    <parent link="base_link"/>
-		    <child link="p3at_back_${suffix}_axle"/>
-	    </joint>
-	    <link name="p3at_back_${suffix}_hub">
-		    <inertial>
-			    <mass value="0.1"/>
-			    <origin xyz="0 0 0"/>
-			    <inertia ixx="1.0" ixy="0.0" ixz="0.0"
-				    iyy="1.0" iyz="0.0" izz="1.0"/>
-  	 	    </inertial>
-	        <visual name="base_visual">
-		        <origin xyz="0 0 0" rpy="0 0 0"/>
-		        <geometry name="pioneer_geom">
-			        <mesh filename="package://p2os_urdf/meshes/p3at_meshes/${suffix}_hubcap.stl"/>
-		        </geometry>
-		        <material name="HubcapYellow"/>
-	        </visual>
-	        <collision>
-		        <origin xyz="0 0 0" rpy="0 0 0"/>
-		        <geometry>
-			        <mesh filename="package://p2os_urdf/meshes/p3at_meshes/${suffix}_hubcap.stl"/>
-		        </geometry>
-	        </collision>
-	    </link>
-	    <gazebo reference="p3at_back_${suffix}_hub">
-		    <material value="Gazebo/Yellow"/>
-	    </gazebo>
-	    <joint name="p3at_back_${suffix}_hub_joint" type="fixed">
-		    <origin xyz="-0 ${reflect*0.041} 0" rpy="0 0 0"/>
-		    <parent link="p3at_back_${suffix}_axle"/>
-		    <child link="p3at_back_${suffix}_hub"/>
-	    </joint>
-	    <link name="p3at_back_${suffix}_wheel">
-		    <inertial>
-			    <mass value="0.5"/>
-			    <origin xyz="0 0 0"/>
-			    <inertia ixx="0.012411765597" ixy="0" ixz="0"
-                    iyy="0.015218160428" iyz="0" izz="0.011763977943"/>
-            </inertial>
-	        <visual name="base_visual">
-		        <origin xyz="0 0 0" rpy="0 0 0"/>
-		        <geometry name="pioneer_geom">
-			        <mesh filename="package://p2os_urdf/meshes/p3at_meshes/wheel.stl"/>
-		        </geometry>
-		        <material name="WheelBlack"/>
-	        </visual>
-	        <collision>
-		        <origin xyz="0 0 0" rpy="${-3.1415927/2} 0 0"/>
-		        <geometry>
-	                <!--mesh filename="package://p2os_urdf/meshes/p3at_meshes/wheel.stl"/-->
-	                <cylinder radius="0.111" length="0.075"/>
-		        </geometry>
-	        </collision>
-	    </link>
-	    <gazebo reference="p3at_back_${suffix}_wheel">
-		    <material value="Gazebo/Black"/>
-	    </gazebo>
-	    <joint name="p3at_back_${suffix}_wheel_joint" type="continuous">
-	        <axis xyz="0 1 0"/>
-            <anchor xyz="0 0 0"/>
-            <limit effort="100" velocity="100" />
-            <joint_properties damping="0.7"/>
-		    <origin xyz="0 0 0" rpy="0 0 0"/>
-		    <parent link="p3at_back_${suffix}_hub"/>
-		<child link="p3at_back_${suffix}_wheel"/>
-	</joint>
+  xmlns:controller="http://playerstage.sourceforge.net/gazebo/xmlschema/#controller"
+  xmlns:interface="http://playerstage.sourceforge.net/gazebo/xmlschema/#interface"
+  xmlns:xacro="http://ros.org/wiki/xacro"
+  >
+  <!-- Chassis -->
+  <xacro:macro name="chassis">
+	  <link name="base_link">
+		  <inertial>
+			  <mass value="10.0"/>
+			  <origin xyz="0 0 0.177"/>
+			  <inertia ixx="0.3338" ixy="0.0" ixz="0.0"
+				  iyy="0.4783" iyz="0.0"
+				  izz="0.3338"/>
+		  </inertial>
+		  <visual name="base_visual">
+			  <origin xyz="0 0 0.177" rpy="0 0 0"/>
+			  <geometry name="pioneer_geom">
+				  <mesh filename="package://p2os_urdf/meshes/p3at_meshes/chassis.stl"/>
+			  </geometry>
+			  <material name="ChassisRed">
+				  <color rgba="0.851 0.0 0.0 1.0"/>
+			  </material>
+		  </visual>
+		  <collision>
+			  <origin xyz="0 0 0.177" rpy="0 0 0"/>
+			  <geometry>
+				  <mesh filename="package://p2os_urdf/meshes/p3at_meshes/chassis.stl"/>
+			  </geometry>
+		  </collision>
+	  </link>
+	  <gazebo reference="base_link">
+		  <material value="Gazebo/Red"/>
+	  </gazebo>
+    <!-- Top -->
+	  <link name="top_plate">
+		  <inertial>
+			  <mass value="0.1"/>
+			  <origin xyz="-0.025 0 -0.223"/>
+			  <inertia ixx="1.0" ixy="0.0" ixz="0.0"
+				  iyy="1.0" iyz="0.0"
+ 				  izz="1.0"/>
+		  </inertial>
+		  <visual name="base_visual">
+			  <origin xyz="0 0 0" rpy="0 0 0"/>
+			  <geometry name="pioneer_geom">
+				  <mesh filename="package://p2os_urdf/meshes/p3at_meshes/top.stl"/>
+			  </geometry>
+			  <material name="TopBlack">
+				  <color rgba="0.038 0.038 0.038 1.0"/>
+			  </material>
+		  </visual>
+		  <collision>
+			  <origin xyz="0 0 0" rpy="0 0 0"/>
+			  <geometry>
+				  <box size="0 0 0"/>
+			  </geometry>
+		  </collision>
+	  </link>
+	  <gazebo reference="top_plate">
+		  <material value="Gazebo/Black"/>
+	  </gazebo>
+	  <joint name="base_top_joint" type="fixed">
+		  <origin xyz="0.003 0 0.274" rpy="0 0 0"/>
+		  <parent link="base_link"/>
+		  <child link="top_plate"/>
+	  </joint>
+    <!-- Front + Back Sonar -->
+	  <link name="front_sonar">
+		  <inertial>
+			  <mass value="0.1"/>
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